File: hardware/6502.sch (KiCad schematic (older format))
At the start: 45 parts, among them J1 JMP, J10 JMP, J14 Conn_01x06_Male, J15 Conn_01x08_Male, J16 Conn_01x16_Male, J2 Conn_01x16_Male, J3 CA, J4 CB, J5 W27c512?, J8 Barrel_Jack_MountingPin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

Commit message: PCB Silkscreen annotations added
Parts:
- J9: symbol Connector:USB_B_Micro -> 6502-rescue:USB_B_Micro-Connector
Changed lines of the file:
@@
 EESchema Schematic File Version 4
-LIBS:6502-cache
 EELAYER 30 0
 EELAYER END
@@
 	10500 1100 10500 975
 $Comp
-L Connector:USB_B_Micro J9
+L 6502-rescue:USB_B_Micro-Connector J9
 U 1 1 61E811F7
 P 9600 1200

Commit message: Wireless nRF24L01+ bootloader added! No more Padauk PMS171b!
Parts:
- removed U1: 74HC00, Package_DIP:DIP-14_W7.62mm, symbol 74xx:74HC00
- added C20, C21: 1uF, Capacitor_SMD:C_0805_2012Metric, symbol Device:C_Small
- added J12: Control_bus, Connector_PinHeader_2.54mm:PinHeader_1x08_P2.54mm_Vertical, symbol Connector:Conn_01x08_Male
- added J13: EzRST, Connector_PinHeader_2.54mm:PinHeader_1x02_P2.54mm_Vertical, symbol Connector:Conn_01x02_Male
- added J17, J18: JMP, Connector_PinHeader_2.54mm:PinHeader_1x02_P2.54mm_Vertical, symbol Connector:Conn_01x02_Male
- added R12: 150k, Resistor_SMD:R_0805_2012Metric, symbol Device:R_Small
- added U1: 74HC14, Package_DIP:DIP-14_W7.62mm, symbol 74xx:74HC14
- added U14: 74HC04, Package_DIP:DIP-14_W7.62mm, symbol 74xx:74HC04
- added U17: 74HC00, Package_DIP:DIP-14_W7.62mm, symbol 74xx:74HC00
- J15: value Conn_01x08_Male -> Data_bus; footprint Connector_PinHeader_2.54mm:PinHeader_1x08_P2.54mm_Vertical -> Connector_PinHeader_2.54mm:PinHeader_2x04_P2.54mm_Vertical; symbol Connector:Conn_01x08_Male -> Connector_Generic:Conn_02x04_Odd_Even
- J16: footprint Connector_PinHeader_2.54mm:PinHeader_1x16_P2.54mm_Vertical -> Connector_PinHeader_2.54mm:PinHeader_2x08_P2.54mm_Vertical
Connections:
- net +5V: now also U1.14 (VCC)
- net A14: now also U17.2
- net A15: now also U14.13
- net GND: now also C20.2, R12.2, U1.7 (GND)
- net ~IO_SEL: now also U17.3
- net ~RES: now also J13.2 (Pin_2), U1.12; no longer R2.2, SW1.2
- net ~ROM_SEL: now also U14.12, U17.1; no longer U5.24 (OE)
- net Ø2: now also J17.1 (Pin_1), U1.1
- net Ø1: now reaches U2.3 (Ø1)
- net Ø1: now also J18.1 (Pin_1), U1.5
- net at D5.2 (A), U4.12 (Q4): now also J12.4 (Pin_4)
- net at D6.2 (A), U4.15 (Q5): now also J12.3 (Pin_3)
- net at D7.2 (A), U4.16 (Q6): now also J12.2 (Pin_2)
- net at D8.2 (A), U4.19 (Q7): now also J12.1 (Pin_1)
- net VEN: now reaches D1.2 (A), U4.2 (Q0)
- net VEN: now also J12.8 (Pin_8)
- net at D2.2 (A), U4.5 (Q1): now also J12.7 (Pin_7)
- net at D3.2 (A), U4.6 (Q2): now also J12.6 (Pin_6)
- net at D4.2 (A), U4.9 (Q3): now also J12.5 (Pin_5)
- new net: C20.1, J13.1 (Pin_1), R2.2, SW1.2, U1.11
- new net: U1.2, U1.3
- new net: U1.6, U1.9
- new net: C21.2, U1.10
- new net: C21.1, R12.1, U1.13
- new net Ø1B: J18.2 (Pin_2), U1.8, U5.24 (OE)
- new net Ø2B: J17.2 (Pin_2), U1.4
- no-connect marks 8 -> 7
Other:
- moved on the sheet: C3, D1, D2, D3, D4, D5, D6, D7, D8, J1, J14, J16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
