File: hardware/ram-vga.sch (KiCad schematic (older format))
At the start: 35 parts, among them J11 Conn_01x04_Male, J12 Conn_01x08_Male, J13 Conn_01x08_Male, J6 DB15_Female_HighDensity, J7 Conn_01x12_Male, U10 74HC245, U11 74HC245, U12 PMS171B-SOP16_150mil, U13 74HC245, U14 74HC04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

Commit message: Wireless nRF24L01+ bootloader added! No more Padauk PMS171b!
Parts:
- removed J12, J13: Conn_01x08_Male, Connector_PinHeader_2.54mm:PinHeader_1x08_P2.54mm_Vertical, symbol Connector:Conn_01x08_Male
- removed R12: R_Pull, Resistor_SMD:R_0805_2012Metric, symbol Device:R_Small
- removed U12: PMS171B-SOP16_150mil, Package_SO:SOIC-16_3.9x9.9mm_P1.27mm, symbol Padauk_IC:PMS171B-SOP16_150mil
- removed U13, U9: 74HC245, Package_DIP:DIP-20_W7.62mm, symbol 74xx:74HC245
- removed unit 6 of U14
- removed unit 4 of U14
- removed unit 1 of U17
- removed U6, U7: 74LS161, Package_DIP:DIP-16_W7.62mm, symbol 74xx:74LS161
- added R13, R14, R15, R16: 2k2, Resistor_SMD:R_0805_2012Metric, symbol Device:R
- added U12: 74HC109, Package_DIP:DIP-16_W7.62mm, symbol 74xx:74LS109
- added U6, U7: 74HC590, Package_DIP:DIP-16_W7.62mm, symbol 74xx:74HC590
- added unit 1 of U8
- added unit 2 of U8
- U17: value 74LS00 -> 74HC00
- U8: value 74LS32 -> 74HC32
Connections:
- net +5V: now also U12.1 (~R), U12.11 (~S), U12.15 (~R), U12.16 (VCC), U12.5 (~S), U6.16 (VCC), U7.16 (VCC)
- net 2Mhz: now also U12.12 (C), U12.4 (C)
- net A12: now also U14.5
- net C0: now also U10.18 (B0), U16.10 (A0), U6.15 (Q0)
- net C1: now also U10.17 (B1), U16.9 (A1), U6.1 (Q1)
- net C10: now also U10.12 (B6), U16.4 (A6), U7.2 (Q2); no longer U18.24 (A9)
- net C11: now also U10.11 (B7), U16.3 (A7), U7.3 (Q3)
- net C12: now also U11.18 (B0), U16.25 (A8), U7.4 (Q4)
- net C13: now also U11.17 (B1), U16.24 (A9), U7.5 (Q5)
- net C14: now also U11.16 (B2), U16.21 (A10), U7.6 (Q6)
- net C15: now also U17.5, U7.7 (Q7)
- net C2: now also U10.16 (B2), U16.8 (A2), U6.2 (Q2)
- net C3: now also U10.15 (B3), U16.7 (A3), U12.14 (J), U6.3 (Q3)
- net C4: now also U10.14 (B4), U16.6 (A4), U6.4 (Q4)
- net C5: now also U10.13 (B5), U16.5 (A5), U6.5 (Q5)
- net C7: now also U18.3 (A7), U12.2 (J), U6.7 (Q7)
- net C8: now also U18.25 (A8), U7.15 (Q0); no longer U18.3 (A7)
- net C9: now also U17.4, U18.24 (A9), U7.1 (Q1); no longer U18.25 (A8)
- net GND: now also R13.1, R15.1, R16.1, U12.8 (GND), U6.12 (~CE), U6.8 (GND), U7.8 (GND)
- net HSYNC: now also U12.10 (Q); no longer U8.8
- net VSYNC: now also U12.6 (Q)
- net ~LDOUTPUT: now also U8.6
- net ~RW: now also U8.2; no longer U14.11
- net Ø2: now also U6.11 (CPC), U6.13 (CPR), U6.14 (~OE), U7.11 (CPC), U7.13 (CPR), U7.14 (~OE); no longer U14.5
- net at C19.1, U20.15 (~CE): now also U14.10
- net at U11.12 (B6), U16.1 (A14), U16.22 (~OE~): now also R13.2
- net at U11.14 (B4), U16.2 (A12): now also R15.2
- net at U11.15 (B3), U16.23 (A11): now also R16.2
- net at U11.13 (B5), U16.26 (A13): now also R14.2
- net at U16.27 (~WE~): now also U8.3; no longer U17.6
- net at U14.6: now also U8.5
- net ~RAM_SEL renamed Ø1
- net Ø1: now also U8.1
- new net: U6.9 (~RCO), U7.12 (~CE)
- new net: U12.13 (~K), U8.8
- new net VEN: U14.11
- new net ~IO_SEL: U8.4
- new net ~VCRST: U12.3 (~K), U17.6, U6.10 (~MRC), U7.10 (~MRC)
- no-connect marks 25 -> 16
Other:
- moved on the sheet: C10, C11, C4, C5, C6, C7, C8, C9, U14C, U14G, U16, U17E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
