File: hardware/6502.kicad_pcb (KiCad board)
At the start: 2 copper layers, 149.9 x 74.9 mm, 141 parts, among them J1 5V, J10 JMP, J11 GPCO, J12 Control_bus, J14 Power, J15 Data_bus, J16 Address bus, J17 USB_A, J2 PORTAB, J20 Interface, J3 CA, J4 CB, J5 W27c512?, J6 DB15_Female_HighDensity, J7 Conn_01x12_Male, J8 5V, J9 USB_B_Micro, SW1 SW_Push, U1 74HC14, U10 74HC245, U11 74HC245, U12 74HC109, U13 74HC74, U14 74HC04, U15 MIC5504-3.3YM5, U16 62256, U17 74HC00, U18 w27C512, U19 74LS161, U2 6502, U20 74HC165, U21 74HC00, U3 6522, U4 74HC273, U5 SST39SF010, U6 74HC590, U7 74HC590, U8 74HC32, U9 NRF24L01_Breakout, Y1 16Mhz

Commit message: Revision 2 published
Parts:
- removed RN1: R_Network08, Resistor_THT:R_Array_SIP9
- added R50: 3k, Resistor_SMD:R_0805_2012Metric, F.Cu at (88.8, 64.8)
- added R51: 3k, Resistor_SMD:R_0805_2012Metric, F.Cu at (90.8, 64.8)
- added R52: 3k, Resistor_SMD:R_0805_2012Metric, F.Cu at (92.8, 64.8)
- added R53: 3k, Resistor_SMD:R_0805_2012Metric, F.Cu at (94.8, 64.8)
- added R54: 3k, Resistor_SMD:R_0805_2012Metric, F.Cu at (96.8, 64.8)
- added R55: 3k, Resistor_SMD:R_0805_2012Metric, F.Cu at (98.8, 64.8)
- added R56: 3k, Resistor_SMD:R_0805_2012Metric, F.Cu at (100.8, 64.8)
- added R57: 3k, Resistor_SMD:R_0805_2012Metric, F.Cu at (102.8, 64.8)
- added R58: 5k1, Resistor_SMD:R_0805_2012Metric, F.Cu at (183.5, 62.1)
- added R59: 5k1, Resistor_SMD:R_0805_2012Metric, F.Cu at (183.5, 58.6)
- added Y2: 16Mhz, Crystal:Crystal_SMD_3225-4Pin_3.2x2.5mm, F.Cu at (196.6, 82.2)
- C1, C2: value 18pF -> 14pF
- C20, C21, R12, R2, R22, R7: moved to F.Cu
- J10: value JMP -> USB
- J6: footprint Connector_Dsub:DSUB-15-HD_Female_Horizontal_P2.29x2.54mm_EdgePinOffset9.40mm-Mountingholes -> Connector_Dsub:DSUB-15-HD_Female_Horizontal_P2.29x1.98mm_EdgePinOffset8.35mm_Housed_MountingHolesOffset10.89mm
- J9: value USB_B_Micro -> USB2.0_16P; footprint Connector_USB:USB_Micro-B_Amphenol_10118194_Horizontal -> Connector_USB:USB_C_Receptacle_HCTL_HC-TYPE-C-16P-01A
- R17, R23, R24, R25: value NC -> 2k2; moved to F.Cu
- R26: footprint Jumper:SolderJumper-2_P1.3mm_Open_RoundedPad1.0x1.5mm -> Jumper:SolderJumper-2_P1.3mm_Bridged_RoundedPad1.0x1.5mm
- R28: footprint Jumper:SolderJumper-2_P1.3mm_Open_RoundedPad1.0x1.5mm -> Jumper:SolderJumper-2_P1.3mm_Bridged_RoundedPad1.0x1.5mm; moved to B.Cu
- R48: footprint Resistor_SMD:R_0805_2012Metric -> Jumper:SolderJumper-2_P1.3mm_Bridged_RoundedPad1.0x1.5mm
- U2: value 6502 -> R6502
- U3: value 6522 -> R6522
- moved C19 22.2 mm to (185.9, 96.3)
- moved C21 18.1 mm to (116.8, 99.2)
- moved R12 17.7 mm to (114.2, 99.2)
- moved C20 17.3 mm to (111.6, 99.2)
- moved R2 16.6 mm to (108.5, 99.1)
- moved R7 9.00 mm to (198.1, 72.3), turned to 180 degrees
- moved R22 7.15 mm to (164.5, 104.0)
- moved R6 4.55 mm to (199.2, 97.3), turned to 90 degrees
- moved R28 3.45 mm to (77.5, 104.8), turned to -90 degrees
- moved Y1 2.65 mm to (196.7, 87.0)
- moved J6 2.60 mm to (196.1, 68.1)
- moved C24 1.33 mm to (182.2, 65.3)
- moved J10 1.31 mm to (175.5, 64.9)
- moved R23 1.11 mm to (142.8, 83.5)
- moved R17 1.11 mm to (148.8, 83.5)
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Connections:
- J10 pad 1: Net-(J10-Pad1) -> Net-(J10-Pin_1)
- J10 pad 2: Net-(J10-Pad1) -> Net-(J10-Pin_2)
- J2 pad 13: Net-(J2-Pad13) -> Net-(J2-Pin_13)
- R28 pad 1: Net-(R28-Pad1) -> GND
- R28 pad 2: GND -> Net-(R28-B)
- R48 pad 1: Net-(J2-Pad13) -> SCL_VGA
- R48 pad 2: SCL_VGA -> Net-(J2-Pin_13)
- U19 pad 10: unconnected-(U19-Pad10) -> +5V
- U2 pad 1: Net-(R28-Pad1) -> Net-(R28-B)
- U3 pad 14: Net-(J2-Pad13) -> Net-(J2-Pin_13)
Routing:
- net Net-(C21-Pad1): track 13.4 -> 36.1 mm, vias 0 -> 1
- net Net-(J2-Pin_13): track 0.00 -> 22.2 mm, vias 0 -> 2
- net Net-(J2-Pad13): track 22.2 -> 0.00 mm, vias 2 -> 0
- net Net-(C21-Pad2): track 10.5 -> 25.3 mm
- net Net-(J9-CC2): track 0.00 -> 10.3 mm
- net Net-(J10-Pad1): track 9.22 -> 0.00 mm
- net Net-(DVEN1-K): track 11.2 -> 1.99 mm
- net Net-(U20-~{CE}): track 20.5 -> 29.5 mm, vias 0 -> 1
- net Net-(U20-Q7): track 34.3 -> 42.9 mm, vias 3 -> 1
- net Net-(J9-CC1): track 0.00 -> 8.51 mm
- net Net-(DVB1-K): track 10.1 -> 2.31 mm
- net CTRL3: track 101.3 -> 93.9 mm, vias 4 -> 6
- net Net-(DVB0-K): track 9.59 -> 2.35 mm
- net +5V: track 728.2 -> 735.4 mm, vias 21 -> 22
- net Net-(DCTRL3-K): track 9.35 -> 2.26 mm
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Other:
- board text added: "ABNielsen.com 6502 SBC Rev 2"
- board text removed: "ABNielsen.com 6502 SBC r1 b4"
